Commit message: Added more launch files

File: urdf/lfl_ur3_ezg_tri_real.urdf.xacro (robot description, xacro)
@@ -34,7 +34,12 @@
 </ezgripper_triple_mount>
 <xacro:include filename="$(find visiondisplay)/urdf/Intel_Realsense_D435.urdf.xacro" />
-<!-- Add the D435_base -->
+<!-- Add the D435 -->
 <D435_base prefix="BMR001" parent_link="BMR001tool0" >
 <origin xyz="0.065 0 -0.13" rpy="0 -0.7 0"/>
 </D435_base>
+<xacro:include filename="$(find visiondisplay)/urdf/Intel_Realsense_L515.urdf.xacro" />
+<!-- Add the L515 -->
+<L515_base prefix="BMR001" parent_link="BMR001_lfl_base" >
+<origin xyz=".2 0 1.75" rpy="0 0 0"/>
+</L515_base>
 </robot>
