Commit message: added compatibility with changes in EZGripper, changes for single gripper

File: minilift_description/urdf/lfl_ur3.urdf.xacro (robot description, xacro)
@@ -2,6 +2,5 @@
 <robot name="minilift" xmlns:xacro="http://ros.org/wiki/xacro">
 <xacro:include filename="$(find minilift_description)/urdf/lfl.urdf.xacro" />
-<xacro:lfl_base prefix="BMR001">
-</xacro:lfl_base>
+<xacro:lfl_base prefix="BMR001"/>
 <xacro:arg name="transmission_hw_interface" default="hardware_interface/PositionJointInterface"/>
 <!-- common stuff -->

File: minilift_description/urdf/lfl_ur3_ezg_sing_real.urdf.xacro (robot description, xacro)
@@ -7,17 +7,19 @@
 <xacro:include filename="$(find ezgripper_description)/urdf/ezgripper_single_mount.urdf.xacro" />
 <!-- Add the gripper -->
-<ezgripper_triple_mount prefix="BMR001" parent_link="BMR001tool0" >
-<origin xyz="${ezgripper_offset_x} ${ezgripper_offset_y} ${ezgripper_offset_z}" rpy="0
-0 0" />
-</ezgripper_triple_mount>
+<xacro:ezgripper_single_mount prefix="BMR001" parent_link="BMR001tool0" activate_control="false" >
+	<origin xyz="${ezgripper_offset_x} ${ezgripper_offset_y} ${ezgripper_offset_z}" rpy="0 0 0"/>
+</xacro:ezgripper_single_mount>
 <xacro:include filename="$(find visiondisplay)/urdf/Intel_Realsense_D435.urdf.xacro" />
 <!-- Add the D435 -->
-<D435_base prefix="BMR001" parent_link="BMR001tool0" >
-<origin xyz="0.065 0 -0.13" rpy="0 -0.7 0"/>
-</D435_base>
+<xacro:D435_base prefix="BMR001" parent_link="BMR001tool0" >
+	<origin xyz="0.065 0 -0.13" rpy="0 -0.7 0"/>
+</xacro:D435_base>
 <xacro:include filename="$(find visiondisplay)/urdf/Intel_Realsense_L515.urdf.xacro" />
 <!-- Add the L515 -->
-<L515_base prefix="BMR001" parent_link="BMR001_lfl_base" >
-<origin xyz=".2 0 1.75" rpy="0 0 0"/>
-</L515_base>
+<xacro:L515_base prefix="BMR001" parent_link="BMR001_lfl_base" >
+	<origin xyz=".2 0 1.75" rpy="0 0 0"/>
+</xacro:L515_base>
+<gazebo>
+	<static>false</static>
+</gazebo>
 </robot>

File: minilift_description/urdf/lfl_ur3_ezg_tri_real.urdf.xacro (robot description, xacro)
@@ -8,6 +8,5 @@
 <!-- Add the gripper -->
 <xacro:ezgripper_triple_mount prefix="BMR001" parent_link="BMR001tool0" >
-    <origin xyz="${ezgripper_offset_x} ${ezgripper_offset_y} ${ezgripper_offset_z}" rpy="0
-    0 0" />
+    <origin xyz="${ezgripper_offset_x} ${ezgripper_offset_y} ${ezgripper_offset_z}" rpy="0 0 0" />
 </xacro:ezgripper_triple_mount>
 <xacro:include filename="$(find visiondisplay)/urdf/Intel_Realsense_D435.urdf.xacro" />

File: minilift_description/urdf/materials.xacro (robot description, xacro)
@@ -12,4 +12,7 @@
   <material name="yellow">
     <color rgba="1.0 1.0 0.0 1.0"/>
+  </material>
+	<material name="grey">
+    <color rgba="0.5 0.5 0.5 1"/>
   </material>
   <material name="dark_grey">
