Commit message: Fixed wheel orientations for rolling in Gazebo and ROS

File: minilift_description/urdf/lfl.urdf.xacro (robot description, xacro)
@@ -6,5 +6,5 @@
     <link name="${prefix}_lfl_base">
       <visual>
-        <origin xyz="0 0 0" rpy="0 0 0"/>
+        <origin xyz="0 0 0.0605" rpy="0 0 0"/>
         <geometry>
           <mesh filename="package://minilift_description/meshes/visual/LFL_xyz.stl"/>
@@ -12,5 +12,5 @@
       </visual>
       <collision>
-        <origin xyz="0 0 0" rpy="0 0 0"/>
+        <origin xyz="0 0 0.0605" rpy="0 0 0"/>
         <geometry>
           <mesh filename="package://minilift_description/meshes/collision/LFL_xyz.stl"/>
@@ -25,5 +25,5 @@
     <link name="${prefix}_lfl_liftplate">
       <visual>
-        <origin xyz="0 0 0" rpy="0 0 0"/>
+        <origin xyz="0 0 0" rpy="0 0 3.14159"/>
         <geometry>
           <mesh filename="package://minilift_description/meshes/visual/LFL_liftplate.stl"/>
@@ -31,5 +31,5 @@
       </visual>
       <collision>
-        <origin xyz="0 0 0" rpy="0 0 0"/>
+        <origin xyz="0 0 0" rpy="0 0 3.14159"/>
         <geometry>
           <mesh filename="package://minilift_description/meshes/collision/LFL_liftplate.stl"/>
@@ -37,18 +37,18 @@
       </collision>
     <inertial>
-      <mass value=".3"/>
+      <mass value="1"/>
       <inertia ixx="0.01" ixy="0.0" ixz="0.0" iyy="0.01" iyz="0.0" izz="0.01"/>
     </inertial>
     </link>
     <joint name="${prefix}_lfl_lift" type="prismatic">
-        <origin rpy="0 0 0" xyz="-0.22 0.0 0.0"/>
-        <parent link="${prefix}_lfl_liftplate"/>
-        <child link="${prefix}_lfl_base"/>
-        <axis xyz="0 0 -1"/>
-        <limit effort="0" lower="0.15" upper="1.5" velocity="0.05"/>
+        <origin rpy="0 0 3.14159" xyz="0.22 0.0 0"/>
+        <parent link="${prefix}_lfl_base"/>
+        <child link="${prefix}_lfl_liftplate"/>
+        <axis xyz="0 0 1"/>
+        <limit effort="0.0" lower="0.15" upper="1.5" velocity="0.05"/>
     </joint>
     <link name="${prefix}_left_wheel_link">
       <visual>
-        <origin xyz="0 -0.2625 0" rpy="1.571 0 0"/>
+        <origin xyz="0 0.0 0" rpy="-1.571 0 0"/>
         <geometry>
           <cylinder length="0.005" radius="0.0605"/>
@@ -56,5 +56,5 @@
       </visual>
       <collision>
-        <origin xyz="0 -0.2625 0" rpy="1.571 0 0"/>
+        <origin xyz="0 0.0 0" rpy="-1.571 0 0"/>
         <geometry>
           <cylinder length="0.005" radius="0.0605"/>
@@ -62,11 +62,11 @@
       </collision>
     <inertial>
-      <mass value=".3"/>
-      <inertia ixx="0.01" ixy="0.0" ixz="0.0" iyy="0.01" iyz="0.0" izz="0.01"/>
+      <mass value="3"/>
+      <inertia ixx="0.01" ixy="0.01" ixz="0.01" iyy="0.01" iyz="0.01" izz="0.01"/>
     </inertial>
     </link>
     <link name="${prefix}_right_wheel_link">
       <visual>
-        <origin xyz="0 0.2625 0" rpy="1.571 0 0"/>
+        <origin xyz="0 0.0 0" rpy="1.571 0 0"/>
         <geometry>
           <cylinder length="0.005" radius="0.0605"/>
@@ -74,5 +74,5 @@
       </visual>
       <collision>
-        <origin xyz="0 0.2625 0" rpy="1.571 0 0"/>
+        <origin xyz="0 0.0 0" rpy="1.571 0 0"/>
         <geometry>
           <cylinder length="0.005" radius="0.0605"/>
@@ -80,17 +80,19 @@
       </collision>
     <inertial>
-      <mass value=".3"/>
-      <inertia ixx="0.01" ixy="0.0" ixz="0.0" iyy="0.01" iyz="0.0" izz="0.01"/>
+      <mass value="3"/>
+      <inertia ixx="0.01" ixy="0.01" ixz="0.01" iyy="0.01" iyz="0.01" izz="0.01"/>
     </inertial>
     </link>
     <joint name="${prefix}_lfl_to_left_wheel" type="continuous">
-        <origin rpy="1.571 0 0" xyz="0 0.0 0.0"/>
+        <origin rpy="0.0 0 0" xyz="0.0 -0.2625 0.06050"/>
         <parent link="${prefix}_lfl_base"/>
         <child link="${prefix}_left_wheel_link"/>
+        <axis xyz="0 1 0"/>
     </joint>
     <joint name="${prefix}_lfl_to_right_wheel" type="continuous">
-        <origin rpy="1.571 0 0" xyz="0 0 0.0"/>
+        <origin rpy="0 0 0" xyz="0.0 0.2625 0.06050"/>
         <parent link="${prefix}_lfl_base"/>
         <child link="${prefix}_right_wheel_link"/>
+        <axis xyz="0 1 0"/>
     </joint>
      <gazebo reference="${prefix}_right_wheel_link">

File: minilift_description/urdf/lfl_ur3.urdf.xacro (robot description, xacro)
@@ -22,5 +22,5 @@
     <parent link="BMR001_lfl_liftplate" />
     <child link = "BMR001base_link" />
-    <origin xyz="0.02 0.0 0.1" rpy="0.0 1.571  0.0" />
+    <origin xyz="-0.02 0.0 0.1" rpy="0.0 -1.571  0.0" />
 </joint>
 <xacro:property name="ezgripper_offset_x" value="0.0" />

Commit message: built hierarchy for lfl, lfl/ur3, lfl/ur3+gripper+realsense

File: minilift_description/urdf/lfl.urdf.xacro (robot description, xacro)
@@ -41,6 +41,6 @@
     </inertial>
     </link>
-    <joint name="${prefix}_lfl_lift" type="prismatic">
-        <origin rpy="0 0 3.14159" xyz="0.22 0.0 0"/>
+    <joint name="${prefix}_lfl_lift" type="fixed">
+        <origin rpy="0 0 3.14159" xyz="0.22 0.0 1"/>
         <parent link="${prefix}_lfl_base"/>
         <child link="${prefix}_lfl_liftplate"/>
@@ -85,5 +85,5 @@
     </link>
     <joint name="${prefix}_lfl_to_left_wheel" type="continuous">
-        <origin rpy="0.0 0 0" xyz="0.0 -0.2625 0.06050"/>
+        <origin rpy="0.0 0 0" xyz="0.0 -0.2625 0.0620"/>
         <parent link="${prefix}_lfl_base"/>
         <child link="${prefix}_left_wheel_link"/>
@@ -91,5 +91,5 @@
     </joint>
     <joint name="${prefix}_lfl_to_right_wheel" type="continuous">
-        <origin rpy="0 0 0" xyz="0.0 0.2625 0.06050"/>
+        <origin rpy="0 0 0" xyz="0.0 0.2625 0.0620"/>
         <parent link="${prefix}_lfl_base"/>
         <child link="${prefix}_right_wheel_link"/>

File: minilift_description/urdf/lfl_ur3.urdf.xacro (robot description, xacro)
@@ -24,12 +24,3 @@
     <origin xyz="-0.02 0.0 0.1" rpy="0.0 -1.571  0.0" />
 </joint>
-<xacro:property name="ezgripper_offset_x" value="0.0" />
-<xacro:property name="ezgripper_offset_y" value="0.0" />
-<xacro:property name="ezgripper_offset_z" value="0.0" />
-<xacro:include filename="$(find ezgripper_description)/urdf/ezgripper_single_mount.urdf.xacro" />
-<!-- Add the gripper -->
-<ezgripper_single_mount prefix="BMR001" parent_link="BMR001tool0" >
-<origin xyz="${ezgripper_offset_x} ${ezgripper_offset_y} ${ezgripper_offset_z}" rpy="0
-0 0" />
-</ezgripper_single_mount>
 </robot>

File: minilift_description/urdf/lfl_ur3_ezg_sing_real.urdf.xacro (robot description, xacro)
@@ -5,5 +5,5 @@
 <xacro:property name="ezgripper_offset_y" value="0.0" />
 <xacro:property name="ezgripper_offset_z" value="0.0" />
-<xacro:include filename="$(find ezgripper_description)/urdf/ezgripper_triple_mount.urdf.xacro" />
+<xacro:include filename="$(find ezgripper_description)/urdf/ezgripper_single_mount.urdf.xacro" />
 <!-- Add the gripper -->
 <ezgripper_triple_mount prefix="BMR001" parent_link="BMR001tool0" >
@@ -19,5 +19,5 @@
 <!-- Add the L515 -->
 <L515_base prefix="BMR001" parent_link="BMR001_lfl_base" >
-<origin xyz=".2 0 1.85" rpy="0 0 0"/>
+<origin xyz=".2 0 1.75" rpy="0 0 0"/>
 </L515_base>
 </robot>

Commit message: Moved gazebo inside xacro and added ${prefix} to wheel joint name

File: minilift_description/urdf/lfl.urdf.xacro (robot description, xacro)
@@ -112,13 +112,12 @@
          <material>Gazebo/Grey</material>
      </gazebo>
-</xacro:macro>
 <gazebo>
-  <plugin name="differential_drive_controller" filename="libgazebo_ros_diff_drive.so">
+  <plugin name="differential_drive_controller" filename="libgazebo_ros_diff_drive.so"  params="prefix">
     <!-- Plugin update rate in Hz -->
     <updateRate>0</updateRate>
     <!-- Name of left joint, defaults to `left_joint` -->
-    <leftJoint>base_link_left_wheel_joint</leftJoint>
+    <leftJoint>${prefix}_left_wheel_link</leftJoint>
     <!-- Name of right joint, defaults to `right_joint` -->
-    <rightJoint>base_link_right_wheel_joint</rightJoint>
+    <rightJoint>${prefix}_right_wheel_link</rightJoint>
     <!-- The distance from the center of one wheel to the other, in meters, defaults to 0.34 m -->
     <wheelSeparation>0.5250</wheelSeparation>
@@ -149,3 +148,4 @@
   </plugin>
 </gazebo>
+</xacro:macro>
 </robot>
