Commit message: updated minilift code with diff-drive plugin, reorganized xacros"

File: minilift_description/urdf/lfl.urdf.xacro (robot description, xacro)
@@ -1,151 +1,213 @@
 <?xml version="1.0" encoding="UTF-8"?>
 <robot name="lfl" xmlns:xacro="http://ros.org/wiki/xacro">
-<!--macro name="lfl" params="*origin"-->
+<xacro:include filename="$(find minilift_description)/urdf/materials.xacro" />
+<xacro:include filename="$(find minilift_description)/urdf/macros.xacro" />
 <xacro:macro name="lfl_base" params="prefix">
-    <!-- links -->
-    <link name="${prefix}_lfl_base">
-      <visual>
-        <origin xyz="0 0 0.0605" rpy="0 0 0"/>
-        <geometry>
-          <mesh filename="package://minilift_description/meshes/visual/LFL_xyz.stl"/>
-        </geometry>
-      </visual>
-      <collision>
-        <origin xyz="0 0 0.0605" rpy="0 0 0"/>
-        <geometry>
-          <mesh filename="package://minilift_description/meshes/collision/LFL_xyz.stl"/>
-        </geometry>
-      </collision>
+  <!-- BASE LINK -->
+  <link name="${prefix}_lfl_base">
+    <visual>
+      <origin xyz="0 0 0.0605" rpy="0 0 0"/>
+      <geometry>
+        <mesh filename="package://minilift_description/meshes/visual/LFL_xyz.stl"/>
+      </geometry>
+      <material name="dark_grey"/>
+    </visual>
+    <collision>
+      <origin xyz="0 0 0.0605" rpy="0 0 0"/>
+      <geometry>
+        <mesh filename="package://minilift_description/meshes/collision/steel_base.stl"/>
+      </geometry>
+    </collision>
+  <inertial>
+    <origin xyz=".15 0 0.2" rpy="0 0 0"/>   <!-- Given -->
+    <mass value="0"/>
+    <inertia ixx="0.2" ixy="0.0" ixz="0.0" iyy="0.01" iyz="0.0" izz="0.01"/>
+  </inertial>
+  </link>
+  <gazebo reference="${prefix}_lfl_base">
+    <material>Gazebo/DarkGrey</material>
+  </gazebo>
+  <!-- LIFTPLATE -->
+  <link name="${prefix}_lfl_liftplate">
+    <visual>
+      <origin xyz="0 0 0" rpy="0 0 3.14159"/>
+      <geometry>
+        <mesh filename="package://minilift_description/meshes/visual/LFL_liftplate.stl"/>
+      </geometry>
+      <material name="dark_grey"/>
+    </visual>
+    <collision>
+      <origin xyz="0 0 0" rpy="0 0 3.14159"/>
+      <geometry>
+        <mesh filename="package://minilift_description/meshes/collision/LFL_liftplate.stl"/>
+      </geometry>
+    </collision>
+  <inertial>
+    <mass value="1"/>
+    <inertia ixx="0.01" ixy="0.0" ixz="0.0" iyy="0.01" iyz="0.0" izz="0.01"/>
+  </inertial>
+  </link>
+  <gazebo reference="${prefix}_lfl_liftplate">
+    <material>Gazebo/DarkGrey</material>
+  </gazebo>
+  <joint name="${prefix}_lfl_lift" type="fixed">
+      <origin rpy="0 0 3.14159" xyz="0.22 0.0 1"/>
+      <parent link="${prefix}_lfl_base"/>
+      <child link="${prefix}_lfl_liftplate"/>
+      <axis xyz="0 0 1"/>
+      <limit effort="0.0" lower="0.15" upper="1.5" velocity="0.05"/>
+  </joint>
+  <!-- LEFT TRACTION WHEEL -->
+  <link name="${prefix}_left_wheel_link">
+    <visual>
+      <origin xyz="0 0.0 0" rpy="-1.571 0 0"/>
+      <geometry>
+        <cylinder length="0.05" radius="0.0605"/>
+      </geometry>
+      <material name="black"/>
+    </visual>
+    <collision>
+      <origin xyz="0 0.0 0" rpy="-1.571 0 0"/>
+      <geometry>
+        <cylinder length="0.05" radius="0.0605"/>
+      </geometry>
+    </collision>
+  <inertial>
+    <mass value="3"/>
+    <xacro:cylinder_inertia m="3" r="0.0605" h="0.05"/>
+  </inertial>
+  </link>
+  <gazebo reference="${prefix}_left_wheel_link">
+    <material>Gazebo/Black</material>
+  </gazebo>
+  <joint name="${prefix}_lfl_to_left_wheel" type="continuous">
+    <origin rpy="0.0 0 0" xyz="0.0 0.2625 0.0620"/>
+    <parent link="${prefix}_lfl_base"/>
+    <child link="${prefix}_left_wheel_link"/>
+    <axis xyz="0 1 0"/>
+  </joint>
+  <!-- RIGHT TRACTION WHEEL -->
+  <link name="${prefix}_right_wheel_link">
+    <visual>
+      <origin xyz="0 0.0 0" rpy="-1.571 0 0"/>
+      <geometry>
+        <cylinder length="0.05" radius="0.0605"/>
+      </geometry>
+      <material name="black"/>
+    </visual>
+    <collision>
+      <origin xyz="0 0.0 0" rpy="-1.571 0 0"/>
+      <geometry>
+        <cylinder length="0.05" radius="0.0605"/>
+      </geometry>
+    </collision>
+  <inertial>
+    <mass value="3"/>
+    <xacro:cylinder_inertia m="3" r="0.0605" h="0.05"/>
+  </inertial>
+  </link>
+  <gazebo reference="${prefix}_right_wheel_link">
+    <material>Gazebo/Black</material>
+  </gazebo>
+  <joint name="${prefix}_lfl_to_right_wheel" type="continuous">
+      <origin rpy="0 0 0" xyz="0.0 -0.2625 0.0620"/>
+      <parent link="${prefix}_lfl_base"/>
+      <child link="${prefix}_right_wheel_link"/>
+      <axis xyz="0 1 0"/>
+  </joint>
+ <!-- LEFT CASTOR WHEEL -->
+  <link name="${prefix}_left_castor_wheel_link">
+    <visual>
+      <origin xyz="0 0.0 0" rpy="1.571 0 0"/>
+      <geometry>
+        <cylinder length="0.038" radius="0.038"/>
+      </geometry>
+      <material name="black"/>
+    </visual>
+    <collision>
+      <origin xyz="0 0.0 0" rpy="1.571 0 0"/>
+      <geometry>
+        <cylinder length="0.038" radius="0.038"/>
+      </geometry>
+    </collision>
     <inertial>
-      <origin xyz=".3 0 0" rpy="0 0 0"/>
-      <mass value="30"/>
-      <inertia ixx="0.2" ixy="0.0" ixz="0.0" iyy="0.01" iyz="0.0" izz="0.01"/>
+      <mass value="1.5"/>
+      <xacro:cylinder_inertia m="1.5" r="0.038" h="0.038"/>
     </inertial>
-    </link>
-    <link name="${prefix}_lfl_liftplate">
-      <visual>
-        <origin xyz="0 0 0" rpy="0 0 3.14159"/>
-        <geometry>
-          <mesh filename="package://minilift_description/meshes/visual/LFL_liftplate.stl"/>
-        </geometry>
-      </visual>
-      <collision>
-        <origin xyz="0 0 0" rpy="0 0 3.14159"/>
-        <geometry>
-          <mesh filename="package://minilift_description/meshes/collision/LFL_liftplate.stl"/>
-        </geometry>
-      </collision>
+  </link>
+  <gazebo reference="${prefix}_left_castor_wheel_link">
+    <mu1 value="0.1"/>
+    <mu2 value="0.1"/>
+    <kp  value="10000000.0" />
+    <kd  value="1.0" />
+    <fdir1 value="1 0 0"/>
+    <material>Gazebo/Black</material>
+  </gazebo>
+  <joint name="${prefix}_lfl_to_left_castor_wheel" type="continuous">
+    <origin rpy="0.0 0 0" xyz="0.65 0.2565 0.0310"/>
+    <parent link="${prefix}_lfl_base"/>
+    <child link="${prefix}_left_castor_wheel_link"/>
+    <axis xyz="0 1 0"/>
+  </joint>
+  <!-- RIGHT CASTOR WHEEL -->
+  <link name="${prefix}_right_castor_wheel_link">
+    <visual>
+      <origin xyz="0 0.0 0" rpy="1.571 0 0"/>
+      <geometry>
+        <cylinder length="0.038" radius="0.038"/>
+      </geometry>
+      <material name="black"/>
+    </visual>
+    <collision>
+      <origin xyz="0 0.0 0" rpy="1.571 0 0"/>
+      <geometry>
+        <cylinder length="0.038" radius="0.038"/>
+      </geometry>
+    </collision>
     <inertial>
-      <mass value="1"/>
-      <inertia ixx="0.01" ixy="0.0" ixz="0.0" iyy="0.01" iyz="0.0" izz="0.01"/>
+      <mass value="1.5"/>
+      <xacro:cylinder_inertia m="1.5" r="0.038" h="0.038"/>
     </inertial>
-    </link>
-    <joint name="${prefix}_lfl_lift" type="fixed">
-        <origin rpy="0 0 3.14159" xyz="0.22 0.0 1"/>
-        <parent link="${prefix}_lfl_base"/>
-        <child link="${prefix}_lfl_liftplate"/>
-        <axis xyz="0 0 1"/>
-        <limit effort="0.0" lower="0.15" upper="1.5" velocity="0.05"/>
-    </joint>
-    <link name="${prefix}_left_wheel_link">
-      <visual>
-        <origin xyz="0 0.0 0" rpy="-1.571 0 0"/>
-        <geometry>
-          <cylinder length="0.005" radius="0.0605"/>
-        </geometry>
-      </visual>
-      <collision>
-        <origin xyz="0 0.0 0" rpy="-1.571 0 0"/>
-        <geometry>
-          <cylinder length="0.005" radius="0.0605"/>
-        </geometry>
-      </collision>
-    <inertial>
-      <mass value="3"/>
-      <inertia ixx="0.01" ixy="0.01" ixz="0.01" iyy="0.01" iyz="0.01" izz="0.01"/>
-    </inertial>
-    </link>
-    <link name="${prefix}_right_wheel_link">
-      <visual>
-        <origin xyz="0 0.0 0" rpy="1.571 0 0"/>
-        <geometry>
-          <cylinder length="0.005" radius="0.0605"/>
-        </geometry>
-      </visual>
-      <collision>
-        <origin xyz="0 0.0 0" rpy="1.571 0 0"/>
-        <geometry>
-          <cylinder length="0.005" radius="0.0605"/>
-        </geometry>
-      </collision>
-    <inertial>
-      <mass value="3"/>
-      <inertia ixx="0.01" ixy="0.01" ixz="0.01" iyy="0.01" iyz="0.01" izz="0.01"/>
-    </inertial>
-    </link>
-    <joint name="${prefix}_lfl_to_left_wheel" type="continuous">
-        <origin rpy="0.0 0 0" xyz="0.0 -0.2625 0.0620"/>
-        <parent link="${prefix}_lfl_base"/>
-        <child link="${prefix}_left_wheel_link"/>
-        <axis xyz="0 1 0"/>
-    </joint>
-    <joint name="${prefix}_lfl_to_right_wheel" type="continuous">
-        <origin rpy="0 0 0" xyz="0.0 0.2625 0.0620"/>
-        <parent link="${prefix}_lfl_base"/>
-        <child link="${prefix}_right_wheel_link"/>
-        <axis xyz="0 1 0"/>
-    </joint>
-     <gazebo reference="${prefix}_right_wheel_link">
-         <mu1 value="1000.0"/>
-         <mu2 value="1000.0"/>
-         <kp value="10000000.0" />
-         <kd value="1.0" />
-         <fdr1 value="0 1 0" />
-         <material>Gazebo/Grey</material>
-     </gazebo>
-     <gazebo reference="${prefix}_left_wheel_link">
-         <mu1 value="1000.0"/>
-         <mu2 value="1000.0"/>
-         <kp value="10000000.0" />
-         <kd value="1.0" />
-         <fdr1 value="0 1 0" />
-         <material>Gazebo/Grey</material>
-     </gazebo>
-<gazebo>
-  <plugin name="differential_drive_controller" filename="libgazebo_ros_diff_drive.so"  params="prefix">
-    <!-- Plugin update rate in Hz -->
-    <updateRate>0</updateRate>
-    <!-- Name of left joint, defaults to `left_joint` -->
-    <leftJoint>${prefix}_left_wheel_link</leftJoint>
-    <!-- Name of right joint, defaults to `right_joint` -->
-    <rightJoint>${prefix}_right_wheel_link</rightJoint>
-    <!-- The distance from the center of one wheel to the other, in meters, defaults to 0.34 m -->
-    <wheelSeparation>0.5250</wheelSeparation>
-    <!-- Diameter of the wheels, in meters, defaults to 0.15 m -->
-    <wheelDiameter>0.1210</wheelDiameter>
-    <!-- Wheel acceleration, in rad/s^2, defaults to 0.0 rad/s^2 -->
-    <wheelAcceleration>1.0</wheelAcceleration>
-    <!-- Maximum torque which the wheels can produce, in Nm, defaults to 5 Nm -->
-    <wheelTorque>20</wheelTorque>
-    <!-- Topic to receive geometry_msgs/Twist message commands, defaults to `cmd_vel` -->
-    <commandTopic>cmd_vel</commandTopic>
-    <!-- Topic to publish nav_msgs/Odometry messages, defaults to `odom` -->
-    <odometryTopic>odom</odometryTopic>
-    <!-- Odometry frame, defaults to `odom` -->
-    <odometryFrame>odom</odometryFrame>
-    <!-- Robot frame to calculate odometry from, defaults to `base_footprint` -->
-    <robotBaseFrame>base_footprint</robotBaseFrame>
-    <!-- Odometry source, 0 for ENCODER, 1 for WORLD, defaults to WORLD -->
-    <odometrySource>1</odometrySource>
-    <!-- Set to true to publish transforms for the wheel links, defaults to false -->
-    <publishWheelTF>false</publishWheelTF>
-    <!-- Set to true to publish transforms for the odometry, defaults to true -->
-    <publishOdom>true</publishOdom>
-    <!-- Set to true to publish sensor_msgs/JointState on /joint_states for the wheel joints, defaults to false -->
-    <publishWheelJointState>false</publishWheelJointState>
-    <!-- Set to true to swap right and left wheels, defaults to true -->
-    <legacyMode>false</legacyMode>
-  </plugin>
-</gazebo>
+  </link>
+  <gazebo reference="${prefix}_right_castor_wheel_link">
+    <mu1 value="0.1"/>
+    <mu2 value="0.1"/>
+    <kp  value="10000000.0" />
+    <kd  value="1.0" />
+    <fdir1 value="1 0 0"/>
+    <material>Gazebo/Black</material>
+  </gazebo>
+  <joint name="${prefix}_lfl_to_right_castor_wheel" type="continuous">
+    <origin rpy="0.0 0 0" xyz="0.65 -0.2565 0.0310"/>
+    <parent link="${prefix}_lfl_base"/>
+    <child link="${prefix}_right_castor_wheel_link"/>
+    <axis xyz="0 1 0"/>
+  </joint>
+<!--......................DIFFERENTIAL DRIVE PLUGIN .....................................-->
+  <gazebo>
+    <plugin name="differential_drive_controller" filename="libgazebo_ros_diff_drive.so">
+      <robotNamespace>/</robotNamespace>
+      <alwaysOn>true</alwaysOn>
+      <updateRate>50</updateRate>
+      <legacyMode>false</legacyMode>
+      <leftJoint>${prefix}_lfl_to_left_wheel</leftJoint>
+      <rightJoint>${prefix}_lfl_to_right_wheel</rightJoint>
+      <wheelSeparation>0.5250</wheelSeparation>
+      <wheelDiameter>0.1210</wheelDiameter>
+      <commandTopic>cmd_vel</commandTopic>
+      <odometryTopic>odom</odometryTopic>
+      <odometryFrame>odom</odometryFrame>
+      <robotBaseFrame>${prefix}_lfl_base</robotBaseFrame>
+      <publishOdomTF>true</publishOdomTF>
+      <publishWheelTF>false</publishWheelTF>
+      <publishWheelJointState>false</publishWheelJointState>
+      <rosDebugLevel>na</rosDebugLevel>
+      <wheelAcceleration>0</wheelAcceleration>
+      <wheelTorque>20</wheelTorque>
+      <odometrySource>world</odometrySource>
+      <publishTf>1</publishTf>
+    </plugin>
+  </gazebo>
+<!-- ................................................................................ -->
 </xacro:macro>
 </robot>

File: minilift_description/urdf/lfl_ur3.urdf.xacro (robot description, xacro)
@@ -1,4 +1,4 @@
 <?xml version="1.0" encoding="UTF-8"?>
-<robot name="lfl_ur3_gripper" xmlns:xacro="http://ros.org/wiki/xacro">
+<robot name="minilift" xmlns:xacro="http://ros.org/wiki/xacro">
 <xacro:include filename="$(find minilift_description)/urdf/lfl.urdf.xacro" />
 <lfl_base prefix="BMR001">

File: minilift_description/urdf/lfl_ur3_ezg_sing_real.urdf.xacro (robot description, xacro)
@@ -1,4 +1,4 @@
 <?xml version="1.0" encoding="UTF-8"?>
-<robot name="lfl_ur3_gripper" xmlns:xacro="http://ros.org/wiki/xacro">
+<robot name="minilift" xmlns:xacro="http://ros.org/wiki/xacro">
 <xacro:include filename="$(find minilift_description)/urdf/lfl_ur3.urdf.xacro" />
 <xacro:property name="ezgripper_offset_x" value="0.0" />

File: minilift_description/urdf/lfl_ur3_ezg_tri_real.urdf.xacro (robot description, xacro)
@@ -1,4 +1,4 @@
 <?xml version="1.0" encoding="UTF-8"?>
-<robot name="lfl_ur3_gripper" xmlns:xacro="http://ros.org/wiki/xacro">
+<robot name="minilift" xmlns:xacro="http://ros.org/wiki/xacro">
 <xacro:include filename="$(find minilift_description)/urdf/lfl_ur3.urdf.xacro" />
 <xacro:property name="ezgripper_offset_x" value="0.0" />
@@ -16,8 +16,10 @@
 <origin xyz="0.065 0 -0.13" rpy="0 -0.7 0"/>
 </D435_base>
-<xacro:include filename="$(find visiondisplay)/urdf/Intel_Realsense_L515.urdf.xacro" />
-<!-- Add the L515 -->
-<L515_base prefix="BMR001" parent_link="BMR001_lfl_base" >
+<!-- Add the Top D435 -->
+<D435_base prefix="BMR001_top" parent_link="BMR001_lfl_base" >
 <origin xyz=".2 0 1.85" rpy="0 0 0"/>
-</L515_base>
+</D435_base>
+<gazebo>
+    <static>false</static>
+</gazebo>
 </robot>

Commit message: added lift controllers

File: minilift_description/urdf/lfl.urdf.xacro (robot description, xacro)
@@ -51,11 +51,23 @@
     <material>Gazebo/DarkGrey</material>
   </gazebo>
-  <joint name="${prefix}_lfl_lift" type="fixed">
+  <joint name="${prefix}_lfl_lift" type="prismatic">
       <origin rpy="0 0 3.14159" xyz="0.22 0.0 1"/>
       <parent link="${prefix}_lfl_base"/>
       <child link="${prefix}_lfl_liftplate"/>
       <axis xyz="0 0 1"/>
-      <limit effort="0.0" lower="0.15" upper="1.5" velocity="0.05"/>
-  </joint>
+      <limit effort="100.0" lower="0.15" upper="0.56" velocity="0.05"/>
+      <dynamics damping="0.5" friction="0.06"/>
+  </joint>
+  <!-- transmissions for Gazebo -->
+  <transmission name="${prefix}_lfl_lift_trans">
+    <type>transmission_interface/SimpleTransmission</type>
+    <joint name="${prefix}_lfl_lift">
+        <hardwareInterface>hardware_interface/PositionJointInterface</hardwareInterface>
+    </joint>
+    <actuator name="${prefix}_lfl_lift_motor">
+        <mechanicalReduction>1</mechanicalReduction>
+        <hardwareInterface>hardware_interface/PositionJointInterface</hardwareInterface>
+    </actuator>
+  </transmission>
   <!-- LEFT TRACTION WHEEL -->
   <link name="${prefix}_left_wheel_link">
@@ -74,6 +86,6 @@
     </collision>
   <inertial>
-    <mass value="3"/>
-    <xacro:cylinder_inertia m="3" r="0.0605" h="0.05"/>
+    <mass value="0.1"/>
+    <xacro:cylinder_inertia m="0.1" r="0.0605" h="0.05"/>
   </inertial>
   </link>
@@ -103,6 +115,6 @@
     </collision>
   <inertial>
-    <mass value="3"/>
-    <xacro:cylinder_inertia m="3" r="0.0605" h="0.05"/>
+    <mass value="0.1"/>
+    <xacro:cylinder_inertia m="0.1" r="0.0605" h="0.05"/>
   </inertial>
   </link>
@@ -132,6 +144,6 @@
     </collision>
     <inertial>
-      <mass value="1.5"/>
-      <xacro:cylinder_inertia m="1.5" r="0.038" h="0.038"/>
+      <mass value="0.1"/>
+      <xacro:cylinder_inertia m="0.1" r="0.038" h="0.038"/>
     </inertial>
   </link>
@@ -166,6 +178,6 @@
     </collision>
     <inertial>
-      <mass value="1.5"/>
-      <xacro:cylinder_inertia m="1.5" r="0.038" h="0.038"/>
+      <mass value="0.1"/>
+      <xacro:cylinder_inertia m="0.1" r="0.038" h="0.038"/>
     </inertial>
   </link>

Commit message: updates to support ROS noetic

File: minilift_description/urdf/lfl.urdf.xacro (robot description, xacro)
@@ -4,4 +4,10 @@
 <xacro:include filename="$(find minilift_description)/urdf/macros.xacro" />
 <xacro:macro name="lfl_base" params="prefix">
+  <!-- BASE FOOTPRINT -->
+  <!-- <link name="${prefix}_lfl_base_footprint"/>
+  <joint name="${prefix}_lfl_base_footprint_joint" type="fixed">
+    <parent link="${prefix}_lfl_base_footprint"/>
+    <child link="${prefix}_lfl_base"/>
+  </joint> -->
   <!-- BASE LINK -->
   <link name="${prefix}_lfl_base">

File: minilift_description/urdf/lfl_ur3.urdf.xacro (robot description, xacro)
@@ -2,6 +2,6 @@
 <robot name="minilift" xmlns:xacro="http://ros.org/wiki/xacro">
 <xacro:include filename="$(find minilift_description)/urdf/lfl.urdf.xacro" />
-<lfl_base prefix="BMR001">
-</lfl_base>
+<xacro:lfl_base prefix="BMR001">
+</xacro:lfl_base>
 <xacro:arg name="transmission_hw_interface" default="hardware_interface/PositionJointInterface"/>
 <!-- common stuff -->
@@ -21,5 +21,5 @@
 <joint name="world_joint" type="fixed" >
     <parent link="BMR001_lfl_liftplate" />
-    <child link = "BMR001base_link" />
+    <child link="BMR001base_link" />
     <origin xyz="-0.02 0.0 0.1" rpy="0.0 -1.571  0.0" />
 </joint>

File: minilift_description/urdf/lfl_ur3_ezg_tri_real.urdf.xacro (robot description, xacro)
@@ -7,17 +7,17 @@
 <xacro:include filename="$(find ezgripper_description)/urdf/ezgripper_triple_mount.urdf.xacro" />
 <!-- Add the gripper -->
-<ezgripper_triple_mount prefix="BMR001" parent_link="BMR001tool0" >
-<origin xyz="${ezgripper_offset_x} ${ezgripper_offset_y} ${ezgripper_offset_z}" rpy="0
-0 0" />
-</ezgripper_triple_mount>
+<xacro:ezgripper_triple_mount prefix="BMR001" parent_link="BMR001tool0" >
+    <origin xyz="${ezgripper_offset_x} ${ezgripper_offset_y} ${ezgripper_offset_z}" rpy="0
+    0 0" />
+</xacro:ezgripper_triple_mount>
 <xacro:include filename="$(find visiondisplay)/urdf/Intel_Realsense_D435.urdf.xacro" />
 <!-- Add the D435 -->
-<D435_base prefix="BMR001" parent_link="BMR001tool0" >
+<xacro:D435_base prefix="BMR001" parent_link="BMR001tool0" >
 <origin xyz="0.065 0 -0.13" rpy="0 -0.7 0"/>
-</D435_base>
+</xacro:D435_base>
 <!-- Add the Top D435 -->
-<D435_base prefix="BMR001_top" parent_link="BMR001_lfl_base" >
+<xacro:D435_base prefix="BMR001_top" parent_link="BMR001_lfl_base" >
 <origin xyz=".2 0 1.85" rpy="0 0 0"/>
-</D435_base>
+</xacro:D435_base>
 <gazebo>
     <static>false</static>
