Commit message: Added libraries necessary for the Pasindu_Sandima design.

File: minilift_description/urdf/lfl.urdf.xacro (robot description, xacro)
@@ -1,38 +1,40 @@
-<?xml version="1.0" encoding="UTF-8"?>
-<robot name="lfl" xmlns:xacro="http://ros.org/wiki/xacro">
-<xacro:include filename="$(find minilift_description)/urdf/materials.xacro" />
-<xacro:include filename="$(find minilift_description)/urdf/macros.xacro" />
+<?xml version="1.0"?>
+<robot  xmlns:xacro="http://ros.org/wiki/xacro"
+        name="lfl" >
 <xacro:macro name="lfl_base" params="prefix">
-  <!-- BASE FOOTPRINT -->
-  <!-- <link name="${prefix}_lfl_base_footprint"/>
-  <joint name="${prefix}_lfl_base_footprint_joint" type="fixed">
-    <parent link="${prefix}_lfl_base_footprint"/>
-    <child link="${prefix}_lfl_base"/>
-  </joint> -->
-  <!-- BASE LINK -->
-  <link name="${prefix}_lfl_base">
-    <visual>
-      <origin xyz="0 0 0.0605" rpy="0 0 0"/>
-      <geometry>
-        <mesh filename="package://minilift_description/meshes/visual/LFL_xyz.stl"/>
-      </geometry>
-      <material name="dark_grey"/>
-    </visual>
-    <collision>
-      <origin xyz="0 0 0.0605" rpy="0 0 0"/>
-      <geometry>
-        <mesh filename="package://minilift_description/meshes/collision/steel_base.stl"/>
-      </geometry>
-    </collision>
-  <inertial>
-    <origin xyz=".15 0 0.2" rpy="0 0 0"/>   <!-- Given -->
-    <mass value="0"/>
-    <inertia ixx="0.2" ixy="0.0" ixz="0.0" iyy="0.01" iyz="0.0" izz="0.01"/>
-  </inertial>
-  </link>
-  <gazebo reference="${prefix}_lfl_base">
-    <material>Gazebo/DarkGrey</material>
-  </gazebo>
-  <!-- LIFTPLATE -->
+    <xacro:include filename="$(find minilift_description)/urdf/caster.urdf.xacro" />
+    <xacro:include filename="$(find minilift_description)/urdf/wheel.urdf.xacro" />
+    <xacro:include filename="$(find minilift_description)/urdf/materials.urdf.xacro" />
+    <xacro:arg name="mesh_enabled" default="false" />
+    <xacro:arg name="robot_namespace" default="/"/>
+    <link   name = "${prefix}_lfl_base">
+        <inertial>
+            <origin xyz="-0.108 0 -0.02579" rpy="0 0 0"/>
+            <mass value="3.978"/>
+            <inertia ixx="0.021858680" ixy="0.0" ixz="0.010020353"
+                    iyy="0.078572349" iyz="-0.0"
+                    izz="0.091971324"/>
+        </inertial>
+        <visual>
+                <origin xyz="0 0 0" rpy="0 0 0" />
+                <geometry>
+                    <mesh filename="package://minilift_description/meshes/visual/LFL_xyz.stl" />
+                </geometry>
+        </visual>
+        <collision>
+                <origin xyz="0 0 0" rpy="0 0 0" />
+                <geometry>
+                    <mesh filename="package://minilift_description/meshes/visual/LFL_xyz.stl" />
+                </geometry>
+        </collision>
+    </link>
+    <link   name =  "${prefix}_base_footprint"/>
+    <joint name = "${prefix}_base_joint"  type = "fixed">
+        <parent link="${prefix}_base_footprint"/>
+        <child link="${prefix}_lfl_base"/>
+        <origin xyz="0.0 0.0 0.09188" rpy="0 0 0" />
+        <axis xyz="0 1 0" rpy="0 0 0" />
+    </joint>
+ <!-- LIFTPLATE -->
   <link name="${prefix}_lfl_liftplate">
     <visual>
@@ -76,156 +78,19 @@
     </actuator>
   </transmission>
-  <!-- LEFT TRACTION WHEEL -->
-  <link name="${prefix}_left_wheel_link">
-    <visual>
-      <origin xyz="0 0.0 0" rpy="-1.571 0 0"/>
-      <geometry>
-        <cylinder length="0.05" radius="0.0605"/>
-      </geometry>
-      <material name="black"/>
-    </visual>
-    <collision>
-      <origin xyz="0 0.0 0" rpy="-1.571 0 0"/>
-      <geometry>
-        <cylinder length="0.05" radius="0.0605"/>
-      </geometry>
-    </collision>
-  <inertial>
-    <mass value="0.1"/>
-    <xacro:cylinder_inertia m="0.1" r="0.0605" h="0.05"/>
-  </inertial>
-  </link>
-  <gazebo reference="${prefix}_left_wheel_link">
-    <material>Gazebo/Black</material>
-  </gazebo>
-  <joint name="${prefix}_lfl_to_left_wheel" type="continuous">
-    <origin rpy="0.0 0 0" xyz="0.0 0.2625 0.0620"/>
-    <parent link="${prefix}_lfl_base"/>
-    <child link="${prefix}_left_wheel_link"/>
-    <axis xyz="0 1 0"/>
-  </joint>
-  <!-- RIGHT TRACTION WHEEL -->
-  <link name="${prefix}_right_wheel_link">
-    <visual>
-      <origin xyz="0 0.0 0" rpy="-1.571 0 0"/>
-      <geometry>
-        <cylinder length="0.05" radius="0.0605"/>
-      </geometry>
-      <material name="black"/>
-    </visual>
-    <collision>
-      <origin xyz="0 0.0 0" rpy="-1.571 0 0"/>
-      <geometry>
-        <cylinder length="0.05" radius="0.0605"/>
-      </geometry>
-    </collision>
-  <inertial>
-    <mass value="0.1"/>
-    <xacro:cylinder_inertia m="0.1" r="0.0605" h="0.05"/>
-  </inertial>
-  </link>
-  <gazebo reference="${prefix}_right_wheel_link">
-    <material>Gazebo/Black</material>
-  </gazebo>
-  <joint name="${prefix}_lfl_to_right_wheel" type="continuous">
-      <origin rpy="0 0 0" xyz="0.0 -0.2625 0.0620"/>
-      <parent link="${prefix}_lfl_base"/>
-      <child link="${prefix}_right_wheel_link"/>
-      <axis xyz="0 1 0"/>
-  </joint>
- <!-- LEFT CASTOR WHEEL -->
-  <link name="${prefix}_left_castor_wheel_link">
-    <visual>
-      <origin xyz="0 0.0 0" rpy="1.571 0 0"/>
-      <geometry>
-        <cylinder length="0.038" radius="0.038"/>
-      </geometry>
-      <material name="black"/>
-    </visual>
-    <collision>
-      <origin xyz="0 0.0 0" rpy="1.571 0 0"/>
-      <geometry>
-        <cylinder length="0.038" radius="0.038"/>
-      </geometry>
-    </collision>
-    <inertial>
-      <mass value="0.1"/>
-      <xacro:cylinder_inertia m="0.1" r="0.038" h="0.038"/>
-    </inertial>
-  </link>
-  <gazebo reference="${prefix}_left_castor_wheel_link">
-    <mu1 value="0.1"/>
-    <mu2 value="0.1"/>
-    <kp  value="10000000.0" />
-    <kd  value="1.0" />
-    <fdir1 value="1 0 0"/>
-    <material>Gazebo/Black</material>
-  </gazebo>
-  <joint name="${prefix}_lfl_to_left_castor_wheel" type="continuous">
-    <origin rpy="0.0 0 0" xyz="0.65 0.2565 0.0310"/>
-    <parent link="${prefix}_lfl_base"/>
-    <child link="${prefix}_left_castor_wheel_link"/>
-    <axis xyz="0 1 0"/>
-  </joint>
-  <!-- RIGHT CASTOR WHEEL -->
-  <link name="${prefix}_right_castor_wheel_link">
-    <visual>
-      <origin xyz="0 0.0 0" rpy="1.571 0 0"/>
-      <geometry>
-        <cylinder length="0.038" radius="0.038"/>
-      </geometry>
-      <material name="black"/>
-    </visual>
-    <collision>
-      <origin xyz="0 0.0 0" rpy="1.571 0 0"/>
-      <geometry>
-        <cylinder length="0.038" radius="0.038"/>
-      </geometry>
-    </collision>
-    <inertial>
-      <mass value="0.1"/>
-      <xacro:cylinder_inertia m="0.1" r="0.038" h="0.038"/>
-    </inertial>
-  </link>
-  <gazebo reference="${prefix}_right_castor_wheel_link">
-    <mu1 value="0.1"/>
-    <mu2 value="0.1"/>
-    <kp  value="10000000.0" />
-    <kd  value="1.0" />
-    <fdir1 value="1 0 0"/>
-    <material>Gazebo/Black</material>
-  </gazebo>
-  <joint name="${prefix}_lfl_to_right_castor_wheel" type="continuous">
-    <origin rpy="0.0 0 0" xyz="0.65 -0.2565 0.0310"/>
-    <parent link="${prefix}_lfl_base"/>
-    <child link="${prefix}_right_castor_wheel_link"/>
-    <axis xyz="0 1 0"/>
-  </joint>
-<!--......................DIFFERENTIAL DRIVE PLUGIN .....................................-->
-  <gazebo>
-    <plugin name="differential_drive_controller" filename="libgazebo_ros_diff_drive.so">
-      <robotNamespace>/</robotNamespace>
-      <alwaysOn>true</alwaysOn>
-      <updateRate>50</updateRate>
-      <legacyMode>false</legacyMode>
-      <leftJoint>${prefix}_lfl_to_left_wheel</leftJoint>
-      <rightJoint>${prefix}_lfl_to_right_wheel</rightJoint>
-      <wheelSeparation>0.5250</wheelSeparation>
-      <wheelDiameter>0.1210</wheelDiameter>
-      <commandTopic>cmd_vel</commandTopic>
-      <odometryTopic>odom</odometryTopic>
-      <odometryFrame>odom</odometryFrame>
-      <robotBaseFrame>${prefix}_lfl_base</robotBaseFrame>
-      <publishOdomTF>true</publishOdomTF>
-      <publishWheelTF>false</publishWheelTF>
-      <publishWheelJointState>false</publishWheelJointState>
-      <rosDebugLevel>na</rosDebugLevel>
-      <wheelAcceleration>0</wheelAcceleration>
-      <wheelTorque>20</wheelTorque>
-      <odometrySource>world</odometrySource>
-      <publishTf>1</publishTf>
-    </plugin>
-  </gazebo>
-<!-- ................................................................................ -->
+    <xacro:caster caster_prefix="rear" parent_link="${prefix}_lfl_base" >
+        <origin xyz="-0.20 0.0 -0.02533" rpy="0 0 0" />
+    </xacro:caster>
+    <xacro:wheel wheel_prefix="left" parent_link="${prefix}_lfl_base" >
+        <origin xyz="-0.04 0.14 -0.045" rpy="0 0 0" />
+    </xacro:wheel>
+    <xacro:wheel wheel_prefix="right" parent_link="${prefix}_lfl_base" >
+        <origin xyz="-0.04 -0.14 -0.045" rpy="0 0 0" />
+    </xacro:wheel>
+    <gazebo>
+        <plugin name="gazebo_ros_control" filename="libgazebo_ros_control.so">
+        <robotNamespace>$(arg robot_namespace)</robotNamespace>
+        <legacyModeNS>true</legacyModeNS>
+        </plugin>
+    </gazebo>
 </xacro:macro>
 </robot>
