Commit message: Removed dependencies on onebot installation.

File: minilift_description/urdf/caster.urdf.xacro (robot description, xacro)
@@ -25,5 +25,5 @@
                 <origin xyz="0 0 0" rpy="${M_PI/2} 0 0" />
 				<geometry>
-					<mesh filename="package://onebot_description/meshes/caswheel.dae" />
+					<mesh filename="package:$(find minilift_description)/meshes/caswheel.dae" />
 				</geometry>
 			</visual>
@@ -46,5 +46,5 @@
 					<origin xyz="0 0 0" rpy="0 0 0" />
 					<geometry>
-						<mesh filename="package://onebot_description/meshes/caster_base2.dae" />
+						<mesh filename="package:$(find minilift_description)/meshes/caster_base2.dae" />
 					</geometry>
 				</xacro:if>

File: minilift_description/urdf/wheel.urdf.xacro (robot description, xacro)
@@ -19,5 +19,5 @@
 					<origin xyz="0 0 0" rpy="0 0 ${M_PI/2}" />
 					<geometry>
-						<mesh filename="package://onebot_description/meshes/wheel.dae" />
+						<mesh filename="package:$(find minilift_description)/meshes/wheel.dae" />
 					</geometry>
 				</xacro:if>

Commit message: Improving minilift operation with Gazebo

File: minilift_description/urdf/caster.urdf.xacro (robot description, xacro)
@@ -25,5 +25,5 @@
                 <origin xyz="0 0 0" rpy="${M_PI/2} 0 0" />
 				<geometry>
-					<mesh filename="package:$(find minilift_description)/meshes/caswheel.dae" />
+					<cylinder length="${caster_wheel_length/2}" radius="${caster_wheel_radius}" />
 				</geometry>
 			</visual>
@@ -43,19 +43,11 @@
 			</inertial>
 			<visual>
-				<xacro:if value="$(arg mesh_enabled)">
-					<origin xyz="0 0 0" rpy="0 0 0" />
-					<geometry>
-						<mesh filename="package:$(find minilift_description)/meshes/caster_base2.dae" />
-					</geometry>
-				</xacro:if>
-				<xacro:unless value="$(arg mesh_enabled)">
-					<origin xyz="0 0 ${-caster_base_length/2}" rpy="0 0 0" />
+					<origin xyz="0 0 ${-caster_base_radius}" rpy="0 0 0" />
 					<geometry>
 						<cylinder length="${caster_base_length}" radius="${caster_base_radius}" />
 					</geometry>
-				</xacro:unless>
 			</visual>
 			<collision>
-				<origin xyz="0 0 ${-caster_base_length/2}" rpy="0 0 0" />
+				<origin xyz="0 0 ${-caster_base_radius}" rpy="0 0 0" />
 				<geometry>
 					<cylinder length="${caster_base_length}" radius="${caster_base_radius}" />

File: minilift_description/urdf/minilift.urdf.xacro (robot description, xacro)
@@ -1,14 +1,15 @@
 <?xml version="1.0"?>
 <robot  xmlns:xacro="http://ros.org/wiki/xacro"
-        name="minilift" >
+        name="minilift"  >
+<xacro:property name="prefix" value="BMR001" />
+<xacro:macro name="minilift" params="prefix" >
     <xacro:include filename="$(find minilift_description)/urdf/caster.urdf.xacro" />
     <xacro:include filename="$(find minilift_description)/urdf/wheel.urdf.xacro" />
     <xacro:include filename="$(find minilift_description)/urdf/materials.urdf.xacro" />
-    <xacro:arg name="mesh_enabled" default="false" />
     <xacro:arg name="robot_namespace" default="/"/>
-    <link   name = "base_link">
+    <link   name = "${prefix}_base_link">
         <inertial>
-            <origin xyz="-0.108 0 -0.02579" rpy="0 0 0"/>
-            <mass value="3.978"/>
+            <origin xyz="0.20 0 0.2" rpy="0 0 0"/>
+            <mass value="30"/>
             <inertia ixx="0.021858680" ixy="0.0" ixz="0.010020353"
                     iyy="0.078572349" iyz="-0.0"
@@ -16,41 +17,31 @@
         </inertial>
         <visual>
-            <xacro:if value="$(arg mesh_enabled)">
                 <origin xyz="0 0 0" rpy="0 0 0" />
                 <geometry>
-                    <mesh filename="package://minilift_description/meshes/visual/LFL_xyz.stl" />
+                    <mesh filename="package://minilift_description/meshes/visual/minilift_xyz.stl" />
                 </geometry>
-            </xacro:if>
-            <xacro:unless value="$(arg mesh_enabled)">
-                <origin xyz="-0.125 0 -0.01" rpy="0 0 0" />
-                <geometry>
-                    <box size="0.25 0.25 0.02" />
-                </geometry>
-                <material name="Blue" />
-            </xacro:unless>
         </visual>
         <collision>
-            <origin xyz="-0.125 0 -0.01" rpy="0 0 0" />
-            <geometry>
-                <box size="0.25 0.25 0.02" />
-            </geometry>
-            <material name="Blue" />
+                <origin xyz="0.350 0 0.9" rpy="0 0 0" />
+                <geometry>
+                    <box size="0.736 0.663 1.8"/>
+                </geometry>
         </collision>
     </link>
-    <link   name =  "base_footprint"/>
-    <joint name = "base_joint"  type = "fixed">
-        <parent link="base_footprint"/>
-        <child link="base_link"/>
+    <link   name =  "${prefix}_base_footprint"/>
+    <joint name = "${prefix}_base_joint"  type = "fixed">
+        <parent link="${prefix}_base_footprint"/>
+        <child link="${prefix}_base_link"/>
         <origin xyz="0.0 0.0 0.09188" rpy="0 0 0" />
         <axis xyz="0 1 0" rpy="0 0 0" />
     </joint>
-    <xacro:caster caster_prefix="rear" parent_link="base_link" >
-        <origin xyz="-0.20 0.0 -0.02533" rpy="0 0 0" />
+    <xacro:caster caster_prefix="rear" parent_link="${prefix}_base_link" >
+        <origin xyz=".70 0.0 0" rpy="0 0 0" />
     </xacro:caster>
-    <xacro:wheel wheel_prefix="left" parent_link="base_link" >
-        <origin xyz="-0.04 0.14 -0.045" rpy="0 0 0" />
+    <xacro:wheel wheel_prefix="left" parent_link="${prefix}_base_link" >
+        <origin xyz="0.0 0.2625 0.0" rpy="0 0 0" />
     </xacro:wheel>
-    <xacro:wheel wheel_prefix="right" parent_link="base_link" >
-        <origin xyz="-0.04 -0.14 -0.045" rpy="0 0 0" />
+    <xacro:wheel wheel_prefix="right" parent_link="${prefix}_base_link" >
+        <origin xyz="0.0 -0.2625 0.0" rpy="0 0 0" />
     </xacro:wheel>
     <gazebo>
@@ -60,3 +51,4 @@
         </plugin>
     </gazebo>
+</xacro:macro>
 </robot>

File: minilift_description/urdf/wheel.urdf.xacro (robot description, xacro)
@@ -10,28 +10,18 @@
 			<inertial>
 				<mass value="0.144" />
-				<origin xyz="0 0 0" />
-				<!-- <inertia  ixx="0.00342579" ixy="0" ixz="0" iyy="0.00644801" iyz="0" izz="0.00342579" /> -->
+				<origin xyz="0 0 0" rpy="${M_PI/2} 0 0" />
 				<inertia  ixx="0.00008929863" ixy="0" ixz="0" iyy="0.000168983" iyz="0" izz="0.00008929863" />
 			</inertial>
 			<visual>
 				<material name="Green"/>
-				<xacro:if value="$(arg mesh_enabled)">
-					<origin xyz="0 0 0" rpy="0 0 ${M_PI/2}" />
-					<geometry>
-						<mesh filename="package:$(find minilift_description)/meshes/wheel.dae" />
-					</geometry>
-				</xacro:if>
-				<xacro:unless value="$(arg mesh_enabled)">
 					<origin xyz="0 0 0" rpy="${M_PI/2} 0 0" />
 					<geometry>
-						<cylinder length="0.02" radius="0.04688" />
+						<cylinder length="0.009" radius="0.061" />
 					</geometry>
-				</xacro:unless>
 			</visual>
 			<collision>
-				<material name="Green"/>
 				<origin xyz="0 0 0" rpy="${M_PI/2} 0 0" />
 				<geometry>
-						<cylinder length="0.02" radius="0.04688" />
+						<cylinder length="0.009" radius="0.061" />
 				</geometry>
 			</collision>
